Commit message: adding pep train pipeline

File: src/mybot_description/urdf/xacro/greenbot_with_camera.xacro (robot description, xacro)
@@ -191,4 +191,57 @@
         </plugin>
     </gazebo>
+    <!-- <gazebo>
+        <plugin name="contact_sensor_plugin" filename="libgazebo_ros_bumper.so">
+            <ros>
+            <namespace>/</namespace>
+            <remapping>~bumper:=/bumper_topic</remapping>
+            </ros>
+            <always_on>true</always_on>
+            <update_rate>50.0</update_rate>
+            <contact>
+            <collision>base_link::collision</collision>
+            </contact>
+        </plugin>
+    </gazebo> -->
+    <joint name="bumper_joint" type="fixed">
+        <origin xyz="1 0 0" rpy="0 0 0"/>
+        <parent link="base_link"/>
+        <child link="bumper_link"/>
+    </joint>
+    <link name="bumper_link">
+        <visual>
+            <origin xyz="0 0 0" rpy="0 0 0"/>
+            <geometry>
+                <box size="0.01 0.1 0.1"/>
+            </geometry>
+        </visual>
+        <collision>
+            <origin xyz="0 0 0" rpy="0 0 0"/>
+            <geometry>
+                <box size="0.01 0.1 0.1"/>
+            </geometry>
+        </collision>
+        <inertial>
+            <mass value="0.1"/>
+            <origin xyz="0 0 0" rpy="0 0 0"/>
+            <inertia ixx="1000" ixy="0" ixz="0" iyy="1000" iyz="0" izz="1000"/>
+        </inertial>
+    </link>
+    <gazebo reference="bumper_link">
+        <sensor type="contact" name="bumper">
+            <always_on>true</always_on>
+            <update_rate>1000.0</update_rate>
+            <visualize>true</visualize>
+            <contact>
+                <!-- Specify the correct collision name for bumper_link -->
+                <collision>base_footprint_fixed_joint_lump__base_link_collision</collision>
+            </contact>
+            <plugin name="gazebo_ros_bumper_controller" filename="libgazebo_ros_bumper.so">
+                <updateRate>100</updateRate>
+                <bumperTopicName>bumper</bumperTopicName>
+                <frameName>base_link</frameName>
+            </plugin>
+        </sensor>
+    </gazebo>
     <greenbot_body/>
 </robot>

File: src/mybot_description/urdf/xacro/sensors/camera.xacro (robot description, xacro)
@@ -32,5 +32,5 @@
                 <always_on>true</always_on>
                 <visualize>true</visualize>
-                <update_rate>30</update_rate>
+                <update_rate>10</update_rate>
                 <camera>
                     <horizontal_fov>1.047</horizontal_fov>
@@ -47,5 +47,5 @@
                 <plugin name="camera_controller" filename="libgazebo_ros_camera.so">
                     <alwaysOn>true</alwaysOn>
-                    <updateRate>30.0</updateRate>
+                    <updateRate>10.0</updateRate>
                     <cameraName>${prefix}</cameraName>
                     <imageTopicName>image_raw</imageTopicName>
